File: First_Board.sch (EAGLE design)
At the start: 32 parts, among them U0 F22X4---DA38, U1 TLC59108PW, U3 A1101, U4 TPS62111RSA

Commit message: Updated to add IR
git-svn-id: file:///p/svn/Projects/Boards/Driveway_Lights@58 1e7840b9-f7c2-db11-b69c-00d0b71b9132
Parts:
- added LED10, LED11, LED12, LED9: (no value), led:LED5MM
- added R13, R14: 10k, rcl:R-US_R0603
- added T1, T2: (no value), zetex:NMOSSOT23
- added U$1, U$2: TSOP39338, opto-vishay:TSOP39338
Connections:
- net N$4 renamed PG
- new net IRLED1: T1.G, U0.21
- new net IRLED2: T2.G, U0.22
- new net IR_IN1: U$1.VO, U0.33
- new net IR_IN2: U$2.VO, U0.34
- new net N$2: LED12.C, R14.2
- new net N$3: LED11.C, LED12.A
- new net N$4: LED10.A, LED9.C
- new net N$5: LED10.C, R13.2
- new net N$6: R13.1, T1.D
- new net N$9: R14.1, T2.D
- net 3.3V: now also LED11.A, LED9.A, U$1.VS, U$2.VS
- net GND: now also T1.S, T2.S, U$1.GND, U$2.GND
Changed lines of the file:
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@@
 <part name="P+1" library="SparkFun" deviceset="3.3V" device=""/>
 <part name="P+2" library="SparkFun" deviceset="3.3V" device=""/>
-<part name="P+3" library="SparkFun" deviceset="3.3V" device=""/>
 <part name="GND8" library="supply1" deviceset="GND" device=""/>
 <part name="R1" library="rcl" deviceset="R-US_" device="R0603" value="47k"/>
@@
 <part name="GND15" library="supply1" deviceset="GND" device=""/>
 <part name="U0" library="TI_MSP430_v16" deviceset="F22X4---DA38" device=""/>
+<part name="LED9" library="led" deviceset="LED" device="5MM"/>
+<part name="LED10" library="led" deviceset="LED" device="5MM"/>
+<part name="LED11" library="led" deviceset="LED" device="5MM"/>
+<part name="LED12" library="led" deviceset="LED" device="5MM"/>
+<part name="R13" library="rcl" deviceset="R-US_" device="R0603" value="10k"/>
+<part name="R14" library="rcl" deviceset="R-US_" device="R0603" value="10k"/>
+<part name="P+3" library="SparkFun" deviceset="3.3V" device=""/>
+<part name="P+4" library="SparkFun" deviceset="3.3V" device=""/>
+<part name="T1" library="zetex" deviceset="NMOSSOT23" device=""/>
+<part name="T2" library="zetex" deviceset="NMOSSOT23" device=""/>
+<part name="GND6" library="supply1" deviceset="GND" device=""/>
+<part name="GND7" library="supply1" deviceset="GND" device=""/>
+<part name="U$1" library="opto-vishay" deviceset="TSOP39338" device=""/>
+<part name="U$2" library="opto-vishay" deviceset="TSOP39338" device=""/>
+<part name="P+7" library="SparkFun" deviceset="3.3V" device=""/>
+<part name="P+8" library="SparkFun" deviceset="3.3V" device=""/>
+<part name="GND16" library="supply1" deviceset="GND" device=""/>
+<part name="GND17" library="supply1" deviceset="GND" device=""/>
 </parts>
 <sheets>
@@
 <instance part="P+1" gate="G$1" x="63.5" y="111.76"/>
 <instance part="P+2" gate="G$1" x="-119.38" y="7.62"/>
-<instance part="P+3" gate="G$1" x="45.72" y="38.1"/>
 <instance part="GND8" gate="1" x="-38.1" y="22.86"/>
 <instance part="R1" gate="G$1" x="-55.88" y="50.8" rot="R90"/>
@@
 <instance part="GND15" gate="1" x="124.46" y="-53.34"/>
 <instance part="U0" gate="G$1" x="5.08" y="-7.62"/>
+<instance part="LED9" gate="G$1" x="-30.48" y="-60.96"/>
+<instance part="LED10" gate="G$1" x="-30.48" y="-73.66"/>
+<instance part="LED11" gate="G$1" x="-10.16" y="-60.96"/>
+<instance part="LED12" gate="G$1" x="-10.16" y="-73.66"/>
+<instance part="R13" gate="G$1" x="-30.48" y="-86.36" rot="R90"/>
+<instance part="R14" gate="G$1" x="-10.16" y="-86.36" rot="R90"/>
+<instance part="P+3" gate="G$1" x="-10.16" y="-50.8"/>
+<instance part="P+4" gate="G$1" x="-30.48" y="-50.8"/>
+<instance part="T1" gate="A" x="-30.48" y="-96.52"/>
+<instance part="T2" gate="A" x="-10.16" y="-96.52"/>
+<instance part="GND6" gate="1" x="-10.16" y="-109.22"/>
+<instance part="GND7" gate="1" x="-30.48" y="-109.22"/>
+<instance part="U$1" gate="G$1" x="25.4" y="-68.58"/>
+<instance part="U$2" gate="G$1" x="25.4" y="-93.98"/>
+<instance part="P+7" gate="G$1" x="40.64" y="-63.5"/>
+<instance part="P+8" gate="G$1" x="38.1" y="-86.36"/>
+<instance part="GND16" gate="1" x="38.1" y="-106.68"/>
+<instance part="GND17" gate="1" x="40.64" y="-76.2"/>
 </instances>
 <busses>
@@
 <wire x1="-25.4" y1="-22.86" x2="-33.02" y2="-22.86" width="0.1524" layer="91"/>
 </segment>
+<segment>
+<pinref part="T1" gate="A" pin="S"/>
+<pinref part="GND7" gate="1" pin="GND"/>
+<wire x1="-30.48" y1="-106.68" x2="-30.48" y2="-101.6" width="0.1524" layer="91"/>
+</segment>
+<segment>
+<pinref part="T2" gate="A" pin="S"/>
+<pinref part="GND6" gate="1" pin="GND"/>
+<wire x1="-10.16" y1="-106.68" x2="-10.16" y2="-101.6" width="0.1524" layer="91"/>
+</segment>
+<segment>
+<pinref part="U$1" gate="G$1" pin="GND"/>
+<pinref part="GND17" gate="1" pin="GND"/>
+<wire x1="40.64" y1="-73.66" x2="38.1" y2="-73.66" width="0.1524" layer="91"/>
+</segment>
+<segment>
+<pinref part="GND16" gate="1" pin="GND"/>
+<pinref part="U$2" gate="G$1" pin="GND"/>
+<wire x1="38.1" y1="-104.14" x2="38.1" y2="-99.06" width="0.1524" layer="91"/>
+</segment>
 </net>
 <net name="VIN" class="0">
@@
 </segment>
 </net>
-<net name="N$4" class="0">
+<net name="PG" class="0">
 <segment>
 <pinref part="U4" gate="G$1" pin="PG"/>
@@
 <wire x1="-25.4" y1="-20.32" x2="-33.02" y2="-20.32" width="0.1524" layer="91"/>
 </segment>
+<segment>
+<pinref part="LED9" gate="G$1" pin="A"/>
+<pinref part="P+4" gate="G$1" pin="3.3V"/>
+<wire x1="-30.48" y1="-50.8" x2="-30.48" y2="-58.42" width="0.1524" layer="91"/>
+</segment>
+<segment>
+<pinref part="LED11" gate="G$1" pin="A"/>
+<pinref part="P+3" gate="G$1" pin="3.3V"/>
+<wire x1="-10.16" y1="-50.8" x2="-10.16" y2="-58.42" width="0.1524" layer="91"/>
+</segment>
+<segment>
+<pinref part="U$1" gate="G$1" pin="VS"/>
+<pinref part="P+7" gate="G$1" pin="3.3V"/>
+<wire x1="40.64" y1="-63.5" x2="38.1" y2="-63.5" width="0.1524" layer="91"/>
+</segment>
+<segment>
+<pinref part="U$2" gate="G$1" pin="VS"/>
+<pinref part="P+8" gate="G$1" pin="3.3V"/>
+<wire x1="38.1" y1="-86.36" x2="38.1" y2="-88.9" width="0.1524" layer="91"/>
+</segment>
 </net>
 <net name="SBWTCK" class="0">
@@
 </segment>
 </net>
+<net name="N$2" class="0">
+<segment>
+<pinref part="LED12" gate="G$1" pin="C"/>
+<pinref part="R14" gate="G$1" pin="2"/>
+<wire x1="-10.16" y1="-81.28" x2="-10.16" y2="-78.74" width="0.1524" layer="91"/>
+</segment>
+</net>
+<net name="N$3" class="0">
+<segment>
+<pinref part="LED11" gate="G$1" pin="C"/>
+<pinref part="LED12" gate="G$1" pin="A"/>
+<wire x1="-10.16" y1="-71.12" x2="-10.16" y2="-66.04" width="0.1524" layer="91"/>
+</segment>
+</net>
+<net name="N$4" class="0">
+<segment>
+<pinref part="LED9" gate="G$1" pin="C"/>
+<pinref part="LED10" gate="G$1" pin="A"/>
+<wire x1="-30.48" y1="-71.12" x2="-30.48" y2="-66.04" width="0.1524" layer="91"/>
+</segment>
+</net>
+<net name="N$5" class="0">
+<segment>
+<pinref part="LED10" gate="G$1" pin="C"/>
+<pinref part="R13" gate="G$1" pin="2"/>
+<wire x1="-30.48" y1="-81.28" x2="-30.48" y2="-78.74" width="0.1524" layer="91"/>
+</segment>
+</net>
+<net name="N$6" class="0">
+<segment>
+<pinref part="R13" gate="G$1" pin="1"/>
+<pinref part="T1" gate="A" pin="D"/>
+</segment>
+</net>
+<net name="N$9" class="0">
+<segment>
+<pinref part="R14" gate="G$1" pin="1"/>
+<pinref part="T2" gate="A" pin="D"/>
+</segment>
+</net>
+<net name="IRLED2" class="0">
+<segment>
+<pinref part="T2" gate="A" pin="G"/>
+<wire x1="-15.24" y1="-99.06" x2="-22.86" y2="-99.06" width="0.1524" layer="91"/>
+</segment>
+<segment>
+<pinref part="U0" gate="G$1" pin="22"/>
+<wire x1="43.18" y1="-25.4" x2="50.8" y2="-25.4" width="0.1524" layer="91"/>
+</segment>
+</net>
+<net name="IRLED1" class="0">
+<segment>
+<pinref part="T1" gate="A" pin="G"/>
+<wire x1="-35.56" y1="-99.06" x2="-45.72" y2="-99.06" width="0.1524" layer="91"/>
+</segment>
+<segment>
+<pinref part="U0" gate="G$1" pin="21"/>
+<wire x1="43.18" y1="-27.94" x2="50.8" y2="-27.94" width="0.1524" layer="91"/>
+</segment>
+</net>
+<net name="IR_IN2" class="0">
+<segment>
+<pinref part="U$2" gate="G$1" pin="VO"/>
+<wire x1="38.1" y1="-93.98" x2="43.18" y2="-93.98" width="0.1524" layer="91"/>
+</segment>
+<segment>
+<pinref part="U0" gate="G$1" pin="34"/>
+<wire x1="43.18" y1="5.08" x2="50.8" y2="5.08" width="0.1524" layer="91"/>
+</segment>
+</net>
+<net name="IR_IN1" class="0">
+<segment>
+<pinref part="U$1" gate="G$1" pin="VO"/>
+<wire x1="38.1" y1="-68.58" x2="45.72" y2="-68.58" width="0.1524" layer="91"/>
+</segment>
+<segment>
+<pinref part="U0" gate="G$1" pin="33"/>
+<wire x1="43.18" y1="2.54" x2="50.8" y2="2.54" width="0.1524" layer="91"/>
+</segment>
+</net>

Commit message: Adding bypass caps
git-svn-id: file:///p/svn/Projects/Boards/Driveway_Lights@59 1e7840b9-f7c2-db11-b69c-00d0b71b9132
Parts:
- added C5, C6, C7: (no value), rcl:C-USC0603
- R13, R14: value 10k -> 10
- renumbered LED10 to IR1A, LED11 to IR2B, LED12 to IR2A, LED9 to IR1B
Connections:
- new net N$11: C6.1, U3.VDCOUP1
- net 3.3V: now also C5.1, C7.1
- net GND: now also C5.2, C6.2, C7.2
Changed lines of the file:
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@@
 <part name="GND15" library="supply1" deviceset="GND" device=""/>
 <part name="U0" library="TI_MSP430_v16" deviceset="F22X4---DA38" device=""/>
-<part name="LED9" library="led" deviceset="LED" device="5MM"/>
-<part name="LED10" library="led" deviceset="LED" device="5MM"/>
-<part name="LED11" library="led" deviceset="LED" device="5MM"/>
-<part name="LED12" library="led" deviceset="LED" device="5MM"/>
-<part name="R13" library="rcl" deviceset="R-US_" device="R0603" value="10k"/>
-<part name="R14" library="rcl" deviceset="R-US_" device="R0603" value="10k"/>
+<part name="IR1B" library="led" deviceset="LED" device="5MM"/>
+<part name="IR1A" library="led" deviceset="LED" device="5MM"/>
+<part name="IR2B" library="led" deviceset="LED" device="5MM"/>
+<part name="IR2A" library="led" deviceset="LED" device="5MM"/>
+<part name="R13" library="rcl" deviceset="R-US_" device="R0603" value="10"/>
+<part name="R14" library="rcl" deviceset="R-US_" device="R0603" value="10"/>
 <part name="P+3" library="SparkFun" deviceset="3.3V" device=""/>
 <part name="P+4" library="SparkFun" deviceset="3.3V" device=""/>
@@
 <part name="GND16" library="supply1" deviceset="GND" device=""/>
 <part name="GND17" library="supply1" deviceset="GND" device=""/>
+<part name="C5" library="rcl" deviceset="C-US" device="C0603"/>
+<part name="C6" library="rcl" deviceset="C-US" device="C0603"/>
+<part name="C7" library="rcl" deviceset="C-US" device="C0603"/>
 </parts>
 <sheets>
@@
 <instance part="GND15" gate="1" x="124.46" y="-53.34"/>
 <instance part="U0" gate="G$1" x="5.08" y="-7.62"/>
-<instance part="LED9" gate="G$1" x="-30.48" y="-60.96"/>
-<instance part="LED10" gate="G$1" x="-30.48" y="-73.66"/>
-<instance part="LED11" gate="G$1" x="-10.16" y="-60.96"/>
-<instance part="LED12" gate="G$1" x="-10.16" y="-73.66"/>
+<instance part="IR1B" gate="G$1" x="-30.48" y="-60.96"/>
+<instance part="IR1A" gate="G$1" x="-30.48" y="-73.66"/>
+<instance part="IR2B" gate="G$1" x="-10.16" y="-60.96"/>
+<instance part="IR2A" gate="G$1" x="-10.16" y="-73.66"/>
 <instance part="R13" gate="G$1" x="-30.48" y="-86.36" rot="R90"/>
 <instance part="R14" gate="G$1" x="-10.16" y="-86.36" rot="R90"/>
@@
 <instance part="GND16" gate="1" x="38.1" y="-106.68"/>
 <instance part="GND17" gate="1" x="40.64" y="-76.2"/>
+<instance part="C5" gate="G$1" x="-48.26" y="10.16"/>
+<instance part="C6" gate="G$1" x="-127" y="-2.54"/>
+<instance part="C7" gate="G$1" x="73.66" y="12.7"/>
 </instances>
 <busses>
@@
 <segment>
 <pinref part="U3" gate="G$1" pin="GND"/>
-<wire x1="-116.84" y1="-15.24" x2="-129.54" y2="-15.24" width="0.1524" layer="91"/>
+<wire x1="-116.84" y1="-15.24" x2="-127" y2="-15.24" width="0.1524" layer="91"/>
+<wire x1="-127" y1="-15.24" x2="-129.54" y2="-15.24" width="0.1524" layer="91"/>
 <wire x1="-129.54" y1="-15.24" x2="-129.54" y2="-22.86" width="0.1524" layer="91"/>
 <pinref part="GND5" gate="1" pin="GND"/>
+<pinref part="C6" gate="G$1" pin="2"/>
+<wire x1="-127" y1="-7.62" x2="-127" y2="-15.24" width="0.1524" layer="91"/>
 </segment>
 <segment>
@@
 <pinref part="U1" gate="G$1" pin="A0"/>
 <wire x1="96.52" y1="0" x2="93.98" y2="0" width="0.1524" layer="91"/>
-<wire x1="93.98" y1="0" x2="81.28" y2="0" width="0.1524" layer="91"/>
+<wire x1="93.98" y1="0" x2="83.82" y2="0" width="0.1524" layer="91"/>
+<wire x1="83.82" y1="0" x2="81.28" y2="0" width="0.1524" layer="91"/>
 <wire x1="81.28" y1="0" x2="81.28" y2="-5.08" width="0.1524" layer="91"/>
 <pinref part="U1" gate="G$1" pin="A1"/>
@@
 <pinref part="U1" gate="G$1" pin="A3"/>
 <wire x1="93.98" y1="7.62" x2="96.52" y2="7.62" width="0.1524" layer="91"/>
+<pinref part="C7" gate="G$1" pin="2"/>
+<wire x1="73.66" y1="7.62" x2="83.82" y2="7.62" width="0.1524" layer="91"/>
+<wire x1="83.82" y1="7.62" x2="83.82" y2="0" width="0.1524" layer="91"/>
 </segment>
 <segment>
@@
 <segment>
 <pinref part="U0" gate="G$1" pin="4"/>
-<wire x1="-25.4" y1="7.62" x2="-33.02" y2="7.62" width="0.1524" layer="91"/>
+<pinref part="C5" gate="G$1" pin="2"/>
+<wire x1="-48.26" y1="5.08" x2="-40.64" y2="5.08" width="0.1524" layer="91"/>
+<wire x1="-40.64" y1="5.08" x2="-40.64" y2="7.62" width="0.1524" layer="91"/>
+<wire x1="-40.64" y1="7.62" x2="-25.4" y2="7.62" width="0.1524" layer="91"/>
 </segment>
 <segment>
@@
 <pinref part="P+6" gate="G$1" pin="3.3V"/>
 <wire x1="91.44" y1="17.78" x2="91.44" y2="22.86" width="0.1524" layer="91"/>
-<wire x1="68.58" y1="17.78" x2="91.44" y2="17.78" width="0.1524" layer="91"/>
+<wire x1="68.58" y1="17.78" x2="73.66" y2="17.78" width="0.1524" layer="91"/>
 <junction x="91.44" y="17.78"/>
+<pinref part="C7" gate="G$1" pin="1"/>
+<wire x1="73.66" y1="17.78" x2="91.44" y2="17.78" width="0.1524" layer="91"/>
+<wire x1="73.66" y1="15.24" x2="73.66" y2="17.78" width="0.1524" layer="91"/>
 </segment>
 <segment>
 <pinref part="U0" gate="G$1" pin="2"/>
-<wire x1="-25.4" y1="12.7" x2="-33.02" y2="12.7" width="0.1524" layer="91"/>
+<pinref part="C5" gate="G$1" pin="1"/>
+<wire x1="-25.4" y1="12.7" x2="-48.26" y2="12.7" width="0.1524" layer="91"/>
 </segment>
 <segment>
@@
 </segment>
 <segment>
-<pinref part="LED9" gate="G$1" pin="A"/>
+<pinref part="IR1B" gate="G$1" pin="A"/>
 <pinref part="P+4" gate="G$1" pin="3.3V"/>
 <wire x1="-30.48" y1="-50.8" x2="-30.48" y2="-58.42" width="0.1524" layer="91"/>
 </segment>
 <segment>
-<pinref part="LED11" gate="G$1" pin="A"/>
+<pinref part="IR2B" gate="G$1" pin="A"/>
 <pinref part="P+3" gate="G$1" pin="3.3V"/>
 <wire x1="-10.16" y1="-50.8" x2="-10.16" y2="-58.42" width="0.1524" layer="91"/>
@@
 <net name="N$2" class="0">
 <segment>
-<pinref part="LED12" gate="G$1" pin="C"/>
+<pinref part="IR2A" gate="G$1" pin="C"/>
 <pinref part="R14" gate="G$1" pin="2"/>
 <wire x1="-10.16" y1="-81.28" x2="-10.16" y2="-78.74" width="0.1524" layer="91"/>
@@
 <net name="N$3" class="0">
 <segment>
-<pinref part="LED11" gate="G$1" pin="C"/>
-<pinref part="LED12" gate="G$1" pin="A"/>
+<pinref part="IR2B" gate="G$1" pin="C"/>
+<pinref part="IR2A" gate="G$1" pin="A"/>
 <wire x1="-10.16" y1="-71.12" x2="-10.16" y2="-66.04" width="0.1524" layer="91"/>
 </segment>
@@
 <net name="N$4" class="0">
 <segment>
-<pinref part="LED9" gate="G$1" pin="C"/>
-<pinref part="LED10" gate="G$1" pin="A"/>
+<pinref part="IR1B" gate="G$1" pin="C"/>
+<pinref part="IR1A" gate="G$1" pin="A"/>
 <wire x1="-30.48" y1="-71.12" x2="-30.48" y2="-66.04" width="0.1524" layer="91"/>
 </segment>
@@
 <net name="N$5" class="0">
 <segment>
-<pinref part="LED10" gate="G$1" pin="C"/>
+<pinref part="IR1A" gate="G$1" pin="C"/>
 <pinref part="R13" gate="G$1" pin="2"/>
 <wire x1="-30.48" y1="-81.28" x2="-30.48" y2="-78.74" width="0.1524" layer="91"/>
@@
 </segment>
 </net>
+<net name="N$11" class="0">
+<segment>
+<pinref part="U3" gate="G$1" pin="VDCOUP1"/>
+<pinref part="C6" gate="G$1" pin="1"/>
+<wire x1="-116.84" y1="0" x2="-127" y2="0" width="0.1524" layer="91"/>
+</segment>
+</net>
